File: kicad/ws2812b-9x9-grid.sch (KiCad schematic (older format))
At the start: 18 parts

Commit message: experimental 9x9-grid board
Parts:
- added P1, P2: CONN_01X03, Connect:PINHEAD1-3, symbol CONN_01X03
- C1, C2, C3, C4, C5, C6, C7, C8, C9: renamed from C?; footprint (none) -> Capacitors_SMD:C_0805_HandSoldering
- D1, D2, D3, D4, D5, D6, D7, D8, D9: renamed from D?; footprint (none) -> ws2812b:WS2812B
Connections:
- net +5V: now also P1.2 (P2), P2.2 (P2)
- net Data_IN: now also P2.3 (P3)
- net Data_OUT: now also P1.3 (P3)
- net GND: now also P1.1 (P1), P2.1 (P1)
Other:
- note added: "Datasheet: https://cdn-shop.adafruit.com/datasheets/WS2812B.pdf"
- moved on the sheet: C1, C2, C3, C4, C5, C6, C7, C8, C9, D1, D2, D3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
