File: kicad/ws2812b-9x9-grid.kicad_pcb (KiCad board)
At the start: 2 copper layers, 24 parts, among them P1 CONN_01X03, P2 CONN_01X03

Commit message: redo layout vdd and gnd planes
Routing:
- net VDD: track 133.5 -> 8.43 mm
- net GND: track 36.3 -> 1.84 mm, vias 20 -> 18
- added copper zone on F.Cu, net VDD
Other:
- board outline added: 49.9 x 25 mm
